Commit message: Add files via upload

File: urdf/ackermann_model.urdf (robot description, URDF)
Before this commit: robot ackermann_model, 9 links, 8 joints
Joints:
- joint left_front_axle: limit (none) -> effort=5 velocity=244
- joint left_rear_axle: limit (none) -> effort=5 velocity=244
- joint left_steering_joint: limit lower=0 upper=0 effort=0 velocity=0 -> lower=-0.4 upper=0.5 effort=0.5 velocity=1
- joint right_front_axle: axis 0 -1 0 -> 0 1 0; limit (none) -> effort=5 velocity=244
- joint right_rear_axle: axis 0 -1 0 -> 0 1 0; limit (none) -> effort=5 velocity=244
- joint right_steering_joint: limit lower=0 upper=0 effort=0 velocity=0 -> lower=-0.4 upper=0.5 effort=0.5 velocity=1
